File: DiffGPS_Hardware/DiffGPS_Hardware.kicad_pcb (KiCad board)
At the start: 2 copper layers, 105.3 x 72.3 mm, 17 parts, among them U1 Raspberry_Pi, U2 OKI

Commit message: Fixed Mistakes from Layout Review
Routing:
- net A3: track 0.00 -> 91.7 mm, vias 0 -> 1
- net +5V: track 15.2 -> 102.2 mm
- net A1: track 0.00 -> 81.9 mm, vias 0 -> 1
- net A2: track 0.00 -> 81.7 mm, vias 0 -> 2
- net VCC: track 0.00 -> 12.0 mm
- net D13: track 0.00 -> 9.41 mm
- net D11: track 0.00 -> 9.41 mm
- net D12: track 0.00 -> 9.41 mm
- net D9: track 0.00 -> 9.26 mm
- net D10: track 0.00 -> 9.26 mm
Changed lines of the file:
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@@
   (segment (start 80.15 100.95) (end 80.15 48.95) (width 0.25) (layer "B.Cu") (net 2))
   (segment (start 84.941 44.073) (end 82.401 44.073) (width 0.508) (layer "F.Cu") (net 5))
+  (segment (start 71.404 61.438) (end 73.66 59.182) (width 0.25) (layer "F.Cu") (net 5))
+  (segment (start 64.262 61.438) (end 71.404 61.438) (width 0.25) (layer "F.Cu") (net 5))
   (segment (start 82.401 44.073) (end 76.5865 49.8875) (width 0.508) (layer "F.Cu") (net 5))
   (segment (start 76.5865 49.8875) (end 72.136 49.8875) (width 0.508) (layer "F.Cu") (net 5))
+  (segment (start 108.11 100.91) (end 106.195 102.825) (width 0.25) (layer "B.Cu") (net 5))
+  (segment (start 79.502 101.327305) (end 79.502 61.468) (width 0.25) (layer "B.Cu") (net 5))
+  (segment (start 77.216 59.182) (end 73.66 59.182) (width 0.25) (layer "B.Cu") (net 5))
+  (segment (start 79.502 61.468) (end 77.216 59.182) (width 0.25) (layer "B.Cu") (net 5))
+  (segment (start 106.195 102.825) (end 80.999695 102.825) (width 0.25) (layer "B.Cu") (net 5))
+  (segment (start 80.999695 102.825) (end 79.502 101.327305) (width 0.25) (layer "B.Cu") (net 5))
   (segment (start 86.434 50.2) (end 90.021 46.613) (width 0.25) (layer "F.Cu") (net 8))
   (segment (start 82.8515 50.2) (end 86.434 50.2) (width 0.25) (layer "F.Cu") (net 8))
@@
   (segment (start 93.85 99.35) (end 95.41 100.91) (width 0.25) (layer "B.Cu") (net 8))
   (segment (start 83.9 99.35) (end 93.85 99.35) (width 0.25) (layer "B.Cu") (net 8))
+  (segment (start 93.995 99.785) (end 119.163 99.785) (width 0.25) (layer "F.Cu") (net 9))
+  (segment (start 92.87 100.91) (end 93.995 99.785) (width 0.25) (layer "F.Cu") (net 9))
+  (segment (start 119.163 99.785) (end 119.634 99.314) (width 0.25) (layer "F.Cu") (net 9))
+  (via (at 119.634 99.314) (size 0.8) (drill 0.4) (layers "F.Cu" "B.Cu") (net 9))
+  (segment (start 120.915 49.567) (end 117.961 46.613) (width 0.25) (layer "B.Cu") (net 9))
+  (segment (start 120.915 98.033) (end 120.915 49.567) (width 0.25) (layer "B.Cu") (net 9))
+  (segment (start 119.634 99.314) (end 120.915 98.033) (width 0.25) (layer "B.Cu") (net 9))
+  (segment (start 117.6015 99.0605) (end 92.1795 99.0605) (width 0.25) (layer "F.Cu") (net 10))
+  (segment (start 118.618 48.768) (end 118.618 48.496) (width 0.25) (layer "F.Cu") (net 10))
+  (segment (start 92.1795 99.0605) (end 90.33 100.91) (width 0.25) (layer "F.Cu") (net 10))
+  (segment (start 118.618 48.496) (end 120.501 46.613) (width 0.25) (layer "F.Cu") (net 10))
+  (segment (start 118.11 98.552) (end 117.6015 99.0605) (width 0.25) (layer "F.Cu") (net 10))
+  (via (at 118.11 98.552) (size 0.8) (drill 0.4) (layers "F.Cu" "B.Cu") (net 10))
+  (via (at 118.618 48.768) (size 0.8) (drill 0.4) (layers "F.Cu" "B.Cu") (net 10))
+  (segment (start 118.618 48.768) (end 118.618 98.044) (width 0.25) (layer "B.Cu") (net 10))
+  (segment (start 118.618 98.044) (end 118.11 98.552) (width 0.25) (layer "B.Cu") (net 10))
+  (segment (start 90.873 97.827) (end 87.79 100.91) (width 0.25) (layer "F.Cu") (net 11))
+  (segment (start 123.317 97.409) (end 122.899 97.827) (width 0.25) (layer "F.Cu") (net 11))
+  (segment (start 122.899 97.827) (end 90.873 97.827) (width 0.25) (layer "F.Cu") (net 11))
+  (via (at 123.317 97.409) (size 0.8) (drill 0.4) (layers "F.Cu" "B.Cu") (net 11))
+  (segment (start 121.676 47.099701) (end 121.676 45.248) (width 0.25) (layer "B.Cu") (net 11))
+  (segment (start 121.676 45.248) (end 120.501 44.073) (width 0.25) (layer "B.Cu") (net 11))
+  (segment (start 123.527701 48.951402) (end 121.676 47.099701) (width 0.25) (layer "B.Cu") (net 11))
+  (segment (start 123.317 97.409) (end 123.527701 97.198299) (width 0.25) (layer "B.Cu") (net 11))
+  (segment (start 123.527701 97.198299) (end 123.527701 48.951402) (width 0.25) (layer "B.Cu") (net 11))
   (segment (start 82.335376 49.1745) (end 84.55 49.1745) (width 0.25) (layer "F.Cu") (net 12))
   (segment (start 81.929461 49.580415) (end 82.335376 49.1745) (width 0.25) (layer "F.Cu") (net 12))
@@
   (segment (start 101.546 45.438) (end 100.181 44.073) (width 0.25) (layer "B.Cu") (net 21))
   (segment (start 101.546 51.594) (end 101.546 45.438) (width 0.25) (layer "B.Cu") (net 21))
+  (segment (start 106.626 45.248) (end 107.801 44.073) (width 0.25) (layer "B.Cu") (net 23))
+  (segment (start 106.626 52.186) (end 106.626 45.248) (width 0.25) (layer "B.Cu") (net 23))
+  (segment (start 107.09 52.65) (end 106.626 52.186) (width 0.25) (layer "B.Cu") (net 23))
+  (segment (start 109.63 52.65) (end 109.166 52.186) (width 0.25) (layer "B.Cu") (net 24))
+  (segment (start 109.166 45.248) (end 110.341 44.073) (width 0.25) (layer "B.Cu") (net 24))
+  (segment (start 109.166 52.186) (end 109.166 45.248) (width 0.25) (layer "B.Cu") (net 24))
+  (segment (start 105.754 47.106) (end 105.261 46.613) (width 0.25) (layer "F.Cu") (net 25))
+  (segment (start 106.626 47.106) (end 105.754 47.106) (width 0.25) (layer "F.Cu") (net 25))
+  (segment (start 112.17 52.65) (end 106.626 47.106) (width 0.25) (layer "F.Cu") (net 25))
+  (segment (start 108.673 46.613) (end 107.801 46.613) (width 0.25) (layer "F.Cu") (net 26))
+  (segment (start 114.71 52.65) (end 108.673 46.613) (width 0.25) (layer "F.Cu") (net 26))
+  (segment (start 117.25 52.65) (end 111.213 46.613) (width 0.25) (layer "F.Cu") (net 27))
+  (segment (start 111.213 46.613) (end 110.341 46.613) (width 0.25) (layer "F.Cu") (net 27))
   (segment (start 70.311 52.9355) (end 68.2885 52.9355) (width 0.508) (layer "F.Cu") (net 31))
   (segment (start 70.311 49.8875) (end 68.2885 49.8875) (width 0.508) (layer "F.Cu") (net 32))
   (segment (start 70.32975 46.8395) (end 68.30725 46.8395) (width 0.25) (layer "F.Cu") (net 33))
+  (segment (start 68.58 59.182) (end 68.58 56.4915) (width 0.25) (layer "F.Cu") (net 34))
+  (segment (start 68.58 56.4915) (end 72.136 52.9355) (width 0.25) (layer "F.Cu") (net 34))
+  (segment (start 64.262 59.182) (end 68.58 59.182) (width 0.25) (layer "F.Cu") (net 34))
   (zone (net 6) (net_name "GND") (layers "F&B.Cu") (hatch edge 0.508)
     (connect_pads yes (clearance 0.127))
