File: DiffGPS_Hardware/DiffGPS_Hardware.kicad_pcb (KiCad board)
At the start: 2 copper layers, 105.3 x 72.3 mm, 17 parts, among them U1 Raspberry_Pi, U2 OKI

Commit message: fixed layout
Parts:
- removed G***: LOGO, MRDT_Silkscreens:0_MRDT_Logo_40mm
- removed G***: LOGO, MRDT_Silkscreens:0_MRDT_Logo_10mm
- A1: moved to B.Cu
- U2: value OKI -> ~; footprint MRDT_Devices:OKI_Horizontal -> SHHD003A04A41:SHHD003A0A-SRZ
- moved A1 48.1 mm to (119.2, 52.8)
- moved U2 24.7 mm to (78.9, 81.6), turned to 90 degrees
- moved C1 7.98 mm to (71.2, 57.7)
- moved C2 7.98 mm to (71.2, 59.9)
- moved H1 4.98 mm to (45.8, 114.2)
- moved H2 4.98 mm to (45.8, 42.0)
Connections:
- Conn1 pad 2: (no net) -> VCC
- U2 pad 3: +5V -> GND
Routing:
- net D13: track 9.41 -> 77.8 mm
- net D12: track 9.41 -> 73.5 mm
- net A0: track 71.5 -> 8.89 mm, vias 1 -> 0
- net D1: track 10.6 -> 71.9 mm
- net D10: track 9.26 -> 70.5 mm, vias 0 -> 1
- net D11: track 9.41 -> 69.6 mm
- net D9: track 9.26 -> 66.4 mm
- net A3: track 91.7 -> 37.4 mm, vias 1 -> 0
- net D2: track 9.81 -> 63.7 mm
- net D3: track 10.6 -> 64.4 mm
- net A1: track 81.9 -> 29.3 mm
- net A4: track 59.3 -> 6.78 mm, vias 2 -> 0
- net D0: track 19.1 -> 71.0 mm, vias 0 -> 1
- net +3V3: track 101.1 -> 49.6 mm, vias 3 -> 2
- net D5: track 6.96 -> 56.4 mm
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Other:
- board size 105.3 x 72.3 mm -> 110.2 x 72.3 mm

Commit message: added mrdt logo
Parts:
- added G***: LOGO, MRDT_Silkscreens:0_MRDT_Logo_30mm, F.Cu at (108.7, 73.6)
Routing:
- net D4: track 75.8 -> 77.3 mm
- net +5V: track 71.5 -> 72.1 mm
