File: DiffGPS_Hardware/DiffGPS_Hardware.kicad_sch (KiCad schematic)
At the start: 15 parts, among them U1 Raspberry_Pi

Commit message: fixed layout
Parts:
- U2: footprint (none) -> SHHD003A04A41:SHHD003A0A-SRZ
Connections:
- net +5V: now also U2.6 (Vout+); no longer U2.4 (Vout+)
- net GND: now also U2.2 (Vin-), U2.3 (On/OFF), U2.4 (Vout-); no longer U2.1 (Vin-), U2.6 (Vout-)
- net VCC: now also U2.1 (Vin+); no longer U2.3 (Vin+)
Changed lines of the file:
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@@
   (junction (at 85.09 104.14) (diameter 0) (color 0 0 0 0)
+  )
+  (junction (at 68.58 30.48) (diameter 0) (color 0 0 0 0)
   )
   (junction (at 16.51 93.98) (diameter 0) (color 0 0 0 0)
@@
     (stroke (width 0) (type default))
   )
+  (wire (pts (xy 68.58 26.67) (xy 68.58 30.48))
+    (stroke (width 0) (type default))
+  )
   (wire (pts (xy 16.51 111.76) (xy 36.83 111.76))
     (stroke (width 0) (type default))
@@
     (stroke (width 0) (type default))
   )
+  (wire (pts (xy 68.58 30.48) (xy 68.58 38.1))
+    (stroke (width 0) (type default))
+  )
   (wire (pts (xy 16.51 73.66) (xy 16.51 93.98))
-    (stroke (width 0) (type default))
-  )
-  (wire (pts (xy 68.58 30.48) (xy 68.58 38.1))
     (stroke (width 0) (type default))
   )
@@
       (effects (font (size 1.27 1.27)))
     )
-    (property "Footprint" "" (at 74.93 35.56 0)
-      (effects (font (size 1.27 1.27)) hide)
-    )
-    (property "Datasheet" "" (at 74.93 35.56 0)
-      (effects (font (size 1.27 1.27)) hide)
-    )
+    (property "Footprint" "SHHD003A04A41:SHHD003A0A-SRZ" (at 74.93 35.56 0)
+      (effects (font (size 1.27 1.27)) hide)
+    )
+    (property "Datasheet" "https://www.digikey.com/en/products/detail/abb-power-conversion/SHHD003A0A41-SRZ/3993519" (at 74.93 35.56 0)
+      (effects (font (size 1.27 1.27)) hide)
+    )

Commit message: updated Pi symbol, fixed various things
Connections:
- net D8: now also U1.18 (GP_24); no longer U1.16 (GP_24)
Changed lines of the file:
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@@
     (pin "15")
     (pin "16")
-    (pin "16")
     (pin "17")
+    (pin "18")
     (pin "19")
     (pin "2")

Commit message: Changed and moved capacitor
Parts:
- C1: footprint Capacitor_SMD:C_0603_1608Metric_Pad1.08x0.95mm_HandSolder -> Capacitor_SMD:C_1206_3216Metric_Pad1.33x1.80mm_HandSolder
- Conn1: footprint MRDT_Connectors:Square_Anderson_2_H_Side_By_Side -> MRDT_Connectors:Square_Anderson_2_H_Side_By_Side_PV
Changed lines of the file:
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@@
       (effects (font (size 1.524 1.524)))
     )
-    (property "Footprint" "MRDT_Connectors:Square_Anderson_2_H_Side_By_Side" (at 15.24 54.61 0)
+    (property "Footprint" "MRDT_Connectors:Square_Anderson_2_H_Side_By_Side_PV" (at 15.24 54.61 0)
       (effects (font (size 1.524 1.524)) hide)
     )
@@
       (effects (font (size 1.524 1.524)))
     )
-    (property "Footprint" "MRDT_Connectors:Square_Anderson_2_H_Side_By_Side" (at 15.24 38.1 0)
+    (property "Footprint" "MRDT_Connectors:Square_Anderson_2_H_Side_By_Side_PV" (at 15.24 38.1 0)
       (effects (font (size 1.524 1.524)) hide)
     )
@@
       (effects (font (size 1.27 1.27)) (justify left))
     )
-    (property "Footprint" "Capacitor_SMD:C_0603_1608Metric_Pad1.08x0.95mm_HandSolder" (at 55.5752 31.75 0)
-      (effects (font (size 1.27 1.27)) hide)
-    )
+    (property "Footprint" "Capacitor_SMD:C_1206_3216Metric_Pad1.33x1.80mm_HandSolder" (at 55.5752 31.75 0)
+      (effects (font (size 1.27 1.27)) hide)
+    )
