File: DiffGPSBreakout/DiffGPSBreakout.kicad_sch (KiCad schematic)
At the start: 15 parts, among them U1 Raspberry_Pi

Commit message: Update DiffGPSBreakout.kicad_sch
Parts:
- U2: footprint SHHD003A04A41:SHHD003A0A-SRZ -> PKE3311PI(P)
Changed lines of the file:
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@@
 			)
 		)
-		(property "Footprint" "SHHD003A04A41:SHHD003A0A-SRZ"
+		(property "Footprint" "PKE3311PI(P)"
 			(at 125.73 54.61 0)
 			(effects
@@
 			)
 		)
-		(property "Datasheet" "https://www.digikey.com/en/products/detail/abb-power-conversion/SHHD003A0A41-SRZ/3993519"
+		(property "Datasheet" "https://flexpowermodules.com/resources/fpm-techspec-pke3000"
 			(at 125.73 54.61 0)
 			(effects
@@
 			)
 		)
-		(property "Description" ""
+		(property "Description" "5V, 6A / 30W"
 			(at 125.73 54.61 0)
 			(effects

Commit message: Changed Schematic Resistor Values
Parts:
- R1: value 3k -> 1.5k
- R2: value 300 -> 220
Changed lines of the file:
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@@
 			)
 		)
-		(property "Value" "3k"
-			(at 68.58 49.53 90)
+		(property "Value" "1.5k"
+			(at 70.104 50.546 0)
 			(effects
 				(font
@@
 		(on_board yes)
 		(dnp no)
-		(fields_autoplaced yes)
 		(property "Reference" "R2"
-			(at 156.718 46.1553 0)
+			(at 156.972 45.72 0)
 			(effects
 				(font
@@
 			)
 		)
-		(property "Value" "300"
-			(at 156.718 48.6922 0)
-			(effects
-				(font
+		(property "Value" "220"
+			(at 156.972 48.26 0)
+			(effects
+				(font
